Commit message: fix: Prepare pre-VLA ROV simulation baseline

File: rospkg/src/kmu26_auv/urdf/rov.urdf (robot description, URDF)
Before this commit: robot rov, 1 links, 0 joints
Links:
- link base_link: geometry collision mesh filename=package://hit25_auv_ros2/meshes/rov_urdf.stl scale=0.001 0.001 0.001; visual mesh filename=package://hit25_auv_ros2/meshes/rov_urdf.stl scale=0.001 0.001 0.001
